Commit message: ready to merge with master

File: rotors_description/urdf/glider_base.xacro (robot description, xacro)
@@ -16,12 +16,5 @@
   <!-- Instantiate fixed wing "mechanics" -->
   <xacro:include filename="$(find rotors_description)/urdf/glider.xacro" />
-  <!-- Mount an ADIS16448 IMU. -->
-  <xacro:default_imu namespace="${namespace}" parent_link="${namespace}/base_link" >
-    <origin xyz="0.3 -0.01 0.023" rpy="0 0 0" />
-  </xacro:default_imu>
-  <!-- Mount a GPS. -->
-  <xacro:default_gps namespace="${namespace}" parent_link="${namespace}/base_link" >
-    <origin xyz="0.22 0 0.143" rpy="0 0 0" />
-  </xacro:default_gps>
+  <!-- ??? - Removing the following breaks aerodynamics -->
   <xacro:default_camera
     namespace="${namespace}"
