Commit message: use wind hack for performance

File: rotors_description/urdf/fixed_wing_X_base.xacro (robot description, xacro)
@@ -67,5 +67,5 @@
       segment_height *axis *joint_origin *inertia_origin *vis_coll_origin *inertia ">
     <xacro:if value="${do_flex}">
-      <joint name="${robot_namespace}/${segment_name}_joint" type="revolute">
+      <joint name="${robot_namespace}/${segment_name}_joint" type="fixed">
         <xacro:insert_block name="joint_origin" />
         <xacro:insert_block name="axis" />
@@ -81,5 +81,5 @@
     </xacro:if>
     <xacro:unless value="${do_flex}">
-      <joint name="${robot_namespace}/${segment_name}_joint" type="revolute">
+      <joint name="${robot_namespace}/${segment_name}_joint" type="fixed">
         <xacro:insert_block name="joint_origin" />
         <xacro:insert_block name="axis" />
@@ -127,5 +127,5 @@
       max_angle color use_mesh_file mesh_file surface_length surface_width
       surface_height *axis *joint_origin *inertia_origin *vis_coll_origin *inertia">
-    <joint name="${robot_namespace}/${surface_name}_joint" type="revolute">
+    <joint name="${robot_namespace}/${surface_name}_joint" type="fixed">
       <xacro:insert_block name="joint_origin" />
       <xacro:insert_block name="axis" />
