Commit message: Modified .yaml and .xacro (David's)

File: rotors_description/urdf/glider.xacro (robot description, xacro)
@@ -24,5 +24,5 @@
   <xacro:property name="PI" value="3.1415926535897931" />
   <!-- Component masses -->
-  <xacro:property name="mass_fuselage" value="3.124" /> <!-- [kg] 3.124-->
+  <xacro:property name="mass_fuselage" value="2.5" /> <!-- [kg] 3.124-->
   <xacro:property name="mass_aileron" value="0.01" /> <!-- [kg] -->
   <xacro:property name="mass_flap" value="0.01" /> <!-- [kg] -->
@@ -112,5 +112,5 @@
     use_mesh_file="${use_mesh}"
     mesh_file="${body_mesh_file}">
-    <origin xyz="0.16 0 0.10" rpy="0 0 0" />
+    <origin xyz="0.13 0 0.10" rpy="0 0 0" />
     <xacro:insert_block name="body_inertia" />
   </xacro:fixed_wing_base_macro>
@@ -313,10 +313,10 @@
       <body>
         <element>
-          <aBdyXX>0.0176</aBdyXX>
-          <aBdyYY>0.0640</aBdyYY>
-          <aBdyZZ>0.0560</aBdyZZ>
-          <forward>1 0 0</forward>
-          <upward>0 0 1</upward>
-          <cp>0.16 0.0 0.05</cp>
+          <aBdyXX>0.002</aBdyXX>
+          <aBdyYY>0.04</aBdyYY>
+          <aBdyZZ>0.04</aBdyZZ>
+          <forward>1 0 0</forward>
+          <upward>0 0 1</upward>
+          <cp>0.13 0.0 0.1</cp>
           <wind name="wind">
             <topic>wind_base_link</topic>
@@ -331,5 +331,5 @@
           <seg_area>0.029</seg_area>
           <seg_chord>0.194</seg_chord>
-          <aeroParamsYAML>${yaml_path}/techpod_TJ_wing.yaml</aeroParamsYAML>
+          <aeroParamsYAML>${yaml_path}/techpod_PLR_wing.yaml</aeroParamsYAML>
           <wind name="wind">
             <topic>wind_base_link</topic>
@@ -342,5 +342,5 @@
           <seg_area>0.042</seg_area>
           <seg_chord>0.183</seg_chord>
-          <aeroParamsYAML>${yaml_path}/techpod_TJ_wing.yaml</aeroParamsYAML>
+          <aeroParamsYAML>${yaml_path}/techpod_PLR_wing.yaml</aeroParamsYAML>
           <wind name="wind">
             <topic>wind_base_link</topic>
@@ -364,5 +364,5 @@
           <seg_area>0.039</seg_area>
           <seg_chord>0.170</seg_chord>
-          <aeroParamsYAML>${yaml_path}/techpod_TJ_wing.yaml</aeroParamsYAML>
+          <aeroParamsYAML>${yaml_path}/techpod_PLR_wing.yaml</aeroParamsYAML>
           <wind name="wind">
             <topic>wind_base_link</topic>
@@ -386,5 +386,5 @@
           <seg_area>0.033</seg_area>
           <seg_chord>0.157</seg_chord>
-          <aeroParamsYAML>${yaml_path}/techpod_TJ_wing.yaml</aeroParamsYAML>
+          <aeroParamsYAML>${yaml_path}/techpod_PLR_wing.yaml</aeroParamsYAML>
           <wind name="wind">
             <topic>wind_base_link</topic>
@@ -397,5 +397,5 @@
           <seg_area>0.026</seg_area>
           <seg_chord>0.146</seg_chord>
-          <aeroParamsYAML>${yaml_path}/techpod_TJ_wing.yaml</aeroParamsYAML>
+          <aeroParamsYAML>${yaml_path}/techpod_PLR_wing.yaml</aeroParamsYAML>
           <wind name="wind">
             <topic>wind_base_link</topic>
@@ -419,5 +419,5 @@
           <seg_area>0.024</seg_area>
           <seg_chord>0.136</seg_chord>
-          <aeroParamsYAML>${yaml_path}/techpod_TJ_wing.yaml</aeroParamsYAML>
+          <aeroParamsYAML>${yaml_path}/techpod_PLR_wing.yaml</aeroParamsYAML>
           <wind name="wind">
             <topic>wind_base_link</topic>
@@ -441,5 +441,5 @@
           <seg_area>0.016</seg_area>
           <seg_chord>0.127</seg_chord>
-          <aeroParamsYAML>${yaml_path}/techpod_TJ_wing.yaml</aeroParamsYAML>
+          <aeroParamsYAML>${yaml_path}/techpod_PLR_wing.yaml</aeroParamsYAML>
           <wind name="wind">
             <topic>wind_base_link</topic>
@@ -452,5 +452,5 @@
           <seg_area>0.029</seg_area>
           <seg_chord>0.194</seg_chord>
-          <aeroParamsYAML>${yaml_path}/techpod_TJ_wing.yaml</aeroParamsYAML>
+          <aeroParamsYAML>${yaml_path}/techpod_PLR_wing.yaml</aeroParamsYAML>
           <wind name="wind">
             <topic>wind_base_link</topic>
@@ -463,5 +463,5 @@
           <seg_area>0.042</seg_area>
           <seg_chord>0.183</seg_chord>
-          <aeroParamsYAML>${yaml_path}/techpod_TJ_wing.yaml</aeroParamsYAML>
+          <aeroParamsYAML>${yaml_path}/techpod_PLR_wing.yaml</aeroParamsYAML>
           <wind name="wind">
             <topic>wind_base_link</topic>
@@ -485,5 +485,5 @@
           <seg_area>0.039</seg_area>
           <seg_chord>0.170</seg_chord>
-          <aeroParamsYAML>${yaml_path}/techpod_TJ_wing.yaml</aeroParamsYAML>
+          <aeroParamsYAML>${yaml_path}/techpod_PLR_wing.yaml</aeroParamsYAML>
           <wind name="wind">
             <topic>wind_base_link</topic>
@@ -507,5 +507,5 @@
           <seg_area>0.033</seg_area>
           <seg_chord>0.157</seg_chord>
-          <aeroParamsYAML>${yaml_path}/techpod_TJ_wing.yaml</aeroParamsYAML>
+          <aeroParamsYAML>${yaml_path}/techpod_PLR_wing.yaml</aeroParamsYAML>
           <wind name="wind">
             <topic>wind_base_link</topic>
@@ -518,5 +518,5 @@
           <seg_area>0.026</seg_area>
           <seg_chord>0.146</seg_chord>
-          <aeroParamsYAML>${yaml_path}/techpod_TJ_wing.yaml</aeroParamsYAML>
+          <aeroParamsYAML>${yaml_path}/techpod_PLR_wing.yaml</aeroParamsYAML>
           <wind name="wind">
             <topic>wind_base_link</topic>
@@ -540,5 +540,5 @@
           <seg_area>0.024</seg_area>
           <seg_chord>0.136</seg_chord>
-          <aeroParamsYAML>${yaml_path}/techpod_TJ_wing.yaml</aeroParamsYAML>
+          <aeroParamsYAML>${yaml_path}/techpod_PLR_wing.yaml</aeroParamsYAML>
           <wind name="wind">
             <topic>wind_base_link</topic>
@@ -562,5 +562,5 @@
           <seg_area>0.016</seg_area>
           <seg_chord>0.127</seg_chord>
-          <aeroParamsYAML>${yaml_path}/techpod_TJ_wing.yaml</aeroParamsYAML>
+          <aeroParamsYAML>${yaml_path}/techpod_PLR_wing.yaml</aeroParamsYAML>
           <wind name="wind">
             <topic>wind_base_link</topic>
@@ -573,5 +573,5 @@
           <seg_area>0.0475</seg_area>
           <seg_chord>0.144</seg_chord>
-          <aeroParamsYAML>${yaml_path}/techpod_TJ_tail_h.yaml</aeroParamsYAML>
+          <aeroParamsYAML>${yaml_path}/techpod_PLR_tail_h.yaml</aeroParamsYAML>
           <indVel name="prop0">
             <topic>prop_slpstr_0</topic>
@@ -598,5 +598,5 @@
           <seg_area>0.0475</seg_area>
           <seg_chord>0.144</seg_chord>
-          <aeroParamsYAML>${yaml_path}/techpod_TJ_tail_h.yaml</aeroParamsYAML>
+          <aeroParamsYAML>${yaml_path}/techpod_PLR_tail_h.yaml</aeroParamsYAML>
           <indVel name="prop0">
             <topic>prop_slpstr_0</topic>
@@ -621,7 +621,8 @@
           <upward>0 -1 0</upward>
           <cp>-0.413 0.0 0.117</cp>
-          <seg_area>0.044</seg_area>
+          <!--<seg_area>0.044</seg_area>-->
+          <seg_area>0.080</seg_area>
           <seg_chord>0.1525</seg_chord>
-          <aeroParamsYAML>${yaml_path}/techpod_TJ_tail_v.yaml</aeroParamsYAML>
+          <aeroParamsYAML>${yaml_path}/techpod_PLR_tail_v.yaml</aeroParamsYAML>
           <indVel name="prop0">
             <topic>prop_slpstr_0</topic>

Commit message: remove prop add ribbon

File: rotors_description/urdf/glider.xacro (robot description, xacro)
@@ -234,5 +234,5 @@
   </xacro:control_surface>
   <!-- Instantiate the propeller -->
-  <xacro:propeller
+  <!-- <xacro:propeller
     robot_namespace="${namespace}"
     suffix="P0"
@@ -244,8 +244,9 @@
     mesh_file="${propeller_mesh_file}">
     <origin xyz="-0.025 0 0.15" rpy="0 ${-0.5*PI} 0" />
-    <origin xyz="-0.1955 0 -0.1672" rpy="0 ${0.5*PI} 0" />   <!-- Mesh origin -->
+    <origin xyz="-0.1955 0 -0.1672" rpy="0 ${0.5*PI} 0" />   Mesh origin
     <xacro:insert_block name="propeller_inertia" />
   </xacro:propeller>
-  <!-- Tracing ribbon/Visual plugin
+-->
+  <!-- Tracing ribbon/Visual plugin -->
   <gazebo reference="${namespace}/base_link">
      <visual>
@@ -253,5 +254,4 @@
      </visual>
   </gazebo>
-  -->
   <xacro:if value="${enable_wind}">
     <gazebo>
